File: symasym/Black_Devil/black_devil/VU-Meter.kicad_sch (KiCad schematic)
At the start: 125 parts, among them J601 Left, J602 Right, J603 Right, U601 LM2902, U602 LM2902, U603 LM2902, U604 LM2902, U605 LM2902, U606 LM2902, U607 LM2902, U608 LM2902

Commit message: VU-Meter Update
added correct values for log scale in 3dB steps
started layout
Parts:
- removed R601, R602, R603, R604, R605, R606, R607, R608, R609, R610, R611, R612, R613, R614, R615, R616, R636, R638, R640, R642, R644, R646, R648, R650, R652, R654, R656, R658, R660, R662, R664, R666: 1k, symbol Device:R
- added R102, R104, R112, R119, R148, R150, R158, R165: 2k2, Resistor_SMD:R_0603_1608Metric, symbol Device:R
- added R103, R149: 39k, Resistor_SMD:R_0603_1608Metric, symbol Device:R
- added R105, R151: 27k, Resistor_SMD:R_0603_1608Metric, symbol Device:R
- added R106, R152: 2k7, Resistor_SMD:R_0603_1608Metric, symbol Device:R
- added R107, R153: 18k, Resistor_SMD:R_0603_1608Metric, symbol Device:R
- added R108, R154: 360, Resistor_SMD:R_0603_1608Metric, symbol Device:R
- added R109, R155: 11k, Resistor_SMD:R_0603_1608Metric, symbol Device:R
- added R110, R116, R118, R156, R162, R164: 390, Resistor_SMD:R_0603_1608Metric, symbol Device:R
- added R111, R157: 10k, Resistor_SMD:R_0603_1608Metric, symbol Device:R
- added R113, R115, R159, R161: 5k1, Resistor_SMD:R_0603_1608Metric, symbol Device:R
- added R114, R120, R124, R160, R166, R170: 100, Resistor_SMD:R_0603_1608Metric, symbol Device:R
- added R117, R163: 3k3, Resistor_SMD:R_0603_1608Metric, symbol Device:R
- added R121, R167: 1k2, Resistor_SMD:R_0603_1608Metric, symbol Device:R
- added R122, R123, R129, R168, R169, R175: 470, Resistor_SMD:R_0603_1608Metric, symbol Device:R
- added R125, R171: 560, Resistor_SMD:R_0603_1608Metric, symbol Device:R
- added R126, R172: 120, Resistor_SMD:R_0603_1608Metric, symbol Device:R
- added R127, R173: 680, Resistor_SMD:R_0603_1608Metric, symbol Device:R
- added R128, R174: 1k8, Resistor_SMD:R_0603_1608Metric, symbol Device:R
- added R130, R176: 330, Resistor_SMD:R_0603_1608Metric, symbol Device:R
- C101: renamed from C605; footprint (none) -> Capacitor_SMD:C_0603_1608Metric
- C102: renamed from C604; footprint (none) -> Capacitor_SMD:C_0603_1608Metric
- C103: renamed from C601; footprint (none) -> Capacitor_SMD:C_0603_1608Metric
- C104: renamed from C603; footprint (none) -> Capacitor_SMD:C_0603_1608Metric
- C105: renamed from C602; footprint (none) -> Capacitor_SMD:C_0603_1608Metric
- C106: renamed from C607; footprint (none) -> Capacitor_SMD:C_0603_1608Metric
- C107: renamed from C608; footprint (none) -> Capacitor_SMD:C_0603_1608Metric
- C108: renamed from C606; footprint (none) -> Capacitor_SMD:C_0603_1608Metric
- C109: renamed from C609; footprint (none) -> Capacitor_SMD:C_0603_1608Metric
- C110: renamed from C610; footprint (none) -> Capacitor_SMD:C_0603_1608Metric
- D102: renamed from D618; footprint (none) -> Diode_SMD:D_MiniMELF
- D103: renamed from D613; footprint (none) -> LED_THT:LED_D3.0mm_Clear
- D104: renamed from D614; footprint (none) -> LED_THT:LED_D3.0mm_Clear
- D105: renamed from D615; footprint (none) -> LED_THT:LED_D3.0mm_Clear
- D106: renamed from D616; footprint (none) -> LED_THT:LED_D3.0mm_Clear
- D107: renamed from D609; footprint (none) -> LED_THT:LED_D3.0mm_Clear
- D108: renamed from D610; footprint (none) -> LED_THT:LED_D3.0mm_Clear
- D109: renamed from D611; footprint (none) -> LED_THT:LED_D3.0mm_Clear
- D110: renamed from D612; footprint (none) -> LED_THT:LED_D3.0mm_Clear
- D111: renamed from D605; footprint (none) -> LED_THT:LED_D3.0mm_Clear
- D112: renamed from D606; footprint (none) -> LED_THT:LED_D3.0mm_Clear
- D113: renamed from D607; footprint (none) -> LED_THT:LED_D3.0mm_Clear
- D114: renamed from D608; footprint (none) -> LED_THT:LED_D3.0mm_Clear
- D115: renamed from D604; footprint (none) -> LED_THT:LED_D3.0mm_Clear
- D116: renamed from D603; footprint (none) -> LED_THT:LED_D3.0mm_Clear
- D117: renamed from D602; footprint (none) -> LED_THT:LED_D3.0mm_Clear
- D118: renamed from D601; footprint (none) -> LED_THT:LED_D3.0mm_Clear
- D120: renamed from D619; footprint (none) -> Diode_SMD:D_MiniMELF
- D121: renamed from D621; footprint (none) -> LED_THT:LED_D3.0mm_Clear
- D122: renamed from D622; footprint (none) -> LED_THT:LED_D3.0mm_Clear
- D123: renamed from D623; footprint (none) -> LED_THT:LED_D3.0mm_Clear
- D124: renamed from D624; footprint (none) -> LED_THT:LED_D3.0mm_Clear
- D125: renamed from D625; footprint (none) -> LED_THT:LED_D3.0mm_Clear
- D126: renamed from D626; footprint (none) -> LED_THT:LED_D3.0mm_Clear
- D127: renamed from D627; footprint (none) -> LED_THT:LED_D3.0mm_Clear
- D128: renamed from D628; footprint (none) -> LED_THT:LED_D3.0mm_Clear
- D129: renamed from D629; footprint (none) -> LED_THT:LED_D3.0mm_Clear
- D130: renamed from D630; footprint (none) -> LED_THT:LED_D3.0mm_Clear
- D131: renamed from D631; footprint (none) -> LED_THT:LED_D3.0mm_Clear
- D132: renamed from D632; footprint (none) -> LED_THT:LED_D3.0mm_Clear
- D133: renamed from D633; footprint (none) -> LED_THT:LED_D3.0mm_Clear
- D134: renamed from D634; footprint (none) -> LED_THT:LED_D3.0mm_Clear
- D135: renamed from D635; footprint (none) -> LED_THT:LED_D3.0mm_Clear
- D136: renamed from D636; footprint (none) -> LED_THT:LED_D3.0mm_Clear
- J101: renamed from J601; footprint (none) -> TerminalBlock:TerminalBlock_bornier-2_P5.08mm
- J102: renamed from J603; footprint (none) -> TerminalBlock:TerminalBlock_bornier-2_P5.08mm
- J103: renamed from J602; footprint (none) -> TerminalBlock:TerminalBlock_bornier-2_P5.08mm
- R101: renamed from R633; footprint (none) -> Resistor_SMD:R_0603_1608Metric
- R131: renamed from R629; footprint (none) -> Resistor_SMD:R_0603_1608Metric
- R132: renamed from R630; footprint (none) -> Resistor_SMD:R_0603_1608Metric
- R133: renamed from R631; footprint (none) -> Resistor_SMD:R_0603_1608Metric
- R134: renamed from R632; footprint (none) -> Resistor_SMD:R_0603_1608Metric
- R135: renamed from R625; footprint (none) -> Resistor_SMD:R_0603_1608Metric
- R136: renamed from R626; footprint (none) -> Resistor_SMD:R_0603_1608Metric
- R137: renamed from R627; footprint (none) -> Resistor_SMD:R_0603_1608Metric
- R138: renamed from R628; footprint (none) -> Resistor_SMD:R_0603_1608Metric
- R139: renamed from R621; footprint (none) -> Resistor_SMD:R_0603_1608Metric
- R140: renamed from R622; footprint (none) -> Resistor_SMD:R_0603_1608Metric
- R141: renamed from R623; footprint (none) -> Resistor_SMD:R_0603_1608Metric
- R142: renamed from R624; footprint (none) -> Resistor_SMD:R_0603_1608Metric
- R143: renamed from R620; footprint (none) -> Resistor_SMD:R_0603_1608Metric
- R144: renamed from R619; footprint (none) -> Resistor_SMD:R_0603_1608Metric
- R145: renamed from R618; footprint (none) -> Resistor_SMD:R_0603_1608Metric
- R146: renamed from R617; footprint (none) -> Resistor_SMD:R_0603_1608Metric
- R147: renamed from R634; footprint (none) -> Resistor_SMD:R_0603_1608Metric
- R177: renamed from R635; footprint (none) -> Resistor_SMD:R_0603_1608Metric
- R178: renamed from R637; footprint (none) -> Resistor_SMD:R_0603_1608Metric
- R179: renamed from R639; footprint (none) -> Resistor_SMD:R_0603_1608Metric
- R180: renamed from R641; footprint (none) -> Resistor_SMD:R_0603_1608Metric
- R181: renamed from R643; footprint (none) -> Resistor_SMD:R_0603_1608Metric
- R182: renamed from R645; footprint (none) -> Resistor_SMD:R_0603_1608Metric
- R183: renamed from R647; footprint (none) -> Resistor_SMD:R_0603_1608Metric
- R184: renamed from R649; footprint (none) -> Resistor_SMD:R_0603_1608Metric
- R185: renamed from R651; footprint (none) -> Resistor_SMD:R_0603_1608Metric
- R186: renamed from R653; footprint (none) -> Resistor_SMD:R_0603_1608Metric
- R187: renamed from R655; footprint (none) -> Resistor_SMD:R_0603_1608Metric
- R188: renamed from R657; footprint (none) -> Resistor_SMD:R_0603_1608Metric
- R189: renamed from R659; footprint (none) -> Resistor_SMD:R_0603_1608Metric
- R190: renamed from R661; footprint (none) -> Resistor_SMD:R_0603_1608Metric
- R191: renamed from R663; footprint (none) -> Resistor_SMD:R_0603_1608Metric
- R192: renamed from R665; footprint (none) -> Resistor_SMD:R_0603_1608Metric
- RV101: renamed from RV601; footprint (none) -> Potentiometer_SMD:Potentiometer_Vishay_TS53YJ_Vertical
- RV102: renamed from RV602; footprint (none) -> Potentiometer_SMD:Potentiometer_Vishay_TS53YJ_Vertical
- U101: renamed from U601; footprint (none) -> Package_SO:TSSOP-14_4.4x5mm_P0.65mm
- U102: renamed from U602; footprint (none) -> Package_SO:TSSOP-14_4.4x5mm_P0.65mm
- U103: renamed from U603; footprint (none) -> Package_SO:TSSOP-14_4.4x5mm_P0.65mm
- U104: renamed from U604; footprint (none) -> Package_SO:TSSOP-14_4.4x5mm_P0.65mm
- U105: renamed from U605; footprint (none) -> Package_SO:TSSOP-14_4.4x5mm_P0.65mm
- U106: renamed from U606; footprint (none) -> Package_SO:TSSOP-14_4.4x5mm_P0.65mm
- U107: renamed from U607; footprint (none) -> Package_SO:TSSOP-14_4.4x5mm_P0.65mm
- U108: renamed from U608; footprint (none) -> Package_SO:TSSOP-14_4.4x5mm_P0.65mm
- renumbered D617 to D101, D620 to D119
Connections:
- net +5VA: now also R102.2, R148.2
- net GND: now also RV101.1, R127.2, R173.2; no longer RV101.3
- net at U108.6 (-): now also R171.2, R175.1
- net at U108.9 (-): now also R175.2, R176.1
- net at U103.6 (-): now also R119.2, R128.1
- net at U102.9 (-): now also R113.2, R114.2
- net at U102.13 (-): now also R115.2, R116.2
- net at U107.13 (-): now also R167.2, R168.2
- net at U108.2 (-): now also R169.2, R170.2
- net at U107.2 (-): now also R163.2, R164.2
- net at U107.6 (-): now also R165.2, R174.1
- net at U103.2 (-): now also R117.2, R118.2
- net at U105.6 (-): now also R149.2, R150.2
- net at U105.9 (-): now also R151.2, R152.2
- net at U106.2 (-): now also R155.2, R156.2
- net at U106.6 (-): now also R157.2, R158.2
- net at U106.13 (-): now also R161.2, R162.2
- net at U107.9 (-): now also R166.2, R174.2
- net at U101.9 (-): now also R105.2, R106.2
- net at U101.13 (-): now also R107.2, R108.2
- net at U106.9 (-): now also R159.2, R160.2
- net at C103.1, R101.2: now also RV101.3; no longer RV101.1
- net at U102.2 (-): now also R109.2, R110.2
- net at U103.13 (-): now also R121.2, R122.2
- net at U101.6 (-): now also R103.2, R104.2
- net at U103.9 (-): now also R120.2, R128.2
- net at U104.9 (-): now also R129.2, R130.1
- net at U104.2 (-): now also R123.2, R124.2
- net at U104.6 (-): now also R125.2, R129.1
- net at U104.13 (-): now also R126.2, R130.2
- net at U105.13 (-): now also R153.2, R154.2
- net at U108.13 (-): now also R172.2, R176.2
- net at U102.6 (-): now also R111.2, R112.2
- new net: R156.1, R157.1
- new net: R150.1, R151.1
- new net: R126.1, R127.1
- new net: R112.1, R113.1
- new net: R152.1, R153.1
- new net: R170.1, R171.1
- new net: R116.1, R117.1
- new net: R160.1, R161.1
- new net: R166.1, R167.1
- new net: R110.1, R111.1
- new net: R104.1, R105.1
- new net: R122.1, R123.1
- new net: R106.1, R107.1
- new net: R162.1, R163.1
- new net: R114.1, R115.1
- new net: R158.1, R159.1
- new net: R148.1, R149.1
- new net: R102.1, R103.1
- new net: R164.1, R165.1
- new net: R118.1, R119.1
- new net: R108.1, R109.1
- new net: R154.1, R155.1
- new net: R120.1, R121.1
- new net: R172.1, R173.1
- new net: R124.1, R125.1
- new net: R168.1, R169.1
