File: Hardware/Black_Devil/Softstart.kicad_pcb (KiCad board)
At the start: 2 copper layers, 280 x 120 mm, 88 parts, among them J101 L1, J102 N, J103 L1_F, J104 N, J105 +45VAC, J106 -45VAC, J107 0V, J108 0V, J109 +63VDC, J110 -63VDC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

Commit message: Major Update
Repo Cleanup
Finished VU Meter PCB
Finalized Softstart PCB
Finalized Channel PCB
Parts:
- added G***: LOGO, eigene:logo, F.Cu at (339.5, 101.5)
- added REF**: Symbol_HighVoltage_Type2_CopperTop_VerySmall, Symbol:Symbol_HighVoltage_Type2_CopperTop_VerySmall, F.Cu at (197.5, 140.5)
- added REF**: OSHW-Logo2_9.8x8mm_SilkScreen, Symbol:OSHW-Logo2_9.8x8mm_SilkScreen, F.Cu at (70.5, 100.8)
- added REF**: WEEE-Logo_5.6x8mm_SilkScreen, Symbol:WEEE-Logo_5.6x8mm_SilkScreen, F.Cu at (199.5, 174.0)
- added REF**: Symbol_HighVoltage_Type2_CopperTop_VerySmall, Symbol:Symbol_HighVoltage_Type2_CopperTop_VerySmall, F.Cu at (212.2, 149.8)
Routing:
- net Net-(J126-Pin_1): track 140.9 -> 0.00 mm
- net Net-(J102-Pin_1): track 140.9 -> 0.00 mm
- net Net-(D117-K): track 85.3 -> 0.00 mm
- net Net-(D101-K): track 85.2 -> 0.00 mm
- net Net-(D117-A): track 91.4 -> 33.3 mm
- net Net-(D102-K): track 55.7 -> 0.00 mm
- net Net-(D101-A): track 88.5 -> 33.5 mm
- net Net-(D118-K): track 53.6 -> 0.00 mm
- net Net-(J123-Pin_1): track 29.0 -> 0.00 mm
- net Net-(J101-Pin_1): track 29.0 -> 0.00 mm
- net Net-(F106-Pad2): track 24.6 -> 0.00 mm
- net Net-(F101-Pad2): track 24.2 -> 0.00 mm
- net Net-(D116-K): track 62.0 -> 59.6 mm
- net Net-(D107-K): track 62.3 -> 60.0 mm
- added copper zone on B.Cu, net Net-(D101-A)
- added copper zone on B.Cu, net Net-(D101-K)
- added copper zone on B.Cu, net Net-(D102-K)
- added copper zone on B.Cu, net Net-(D117-A)
- added copper zone on B.Cu, net Net-(D117-K)
- added copper zone on B.Cu, net Net-(D118-K)
- added copper zone on B.Cu, net Net-(F101-Pad2)
- added copper zone on B.Cu, net Net-(F106-Pad2)
- added copper zone on B.Cu, net Net-(J101-Pin_1)
- added copper zone on B.Cu, net Net-(J102-Pin_1)
- added copper zone on B.Cu, net Net-(J123-Pin_1)
- added copper zone on B.Cu, net Net-(J126-Pin_1)
Other:
- board text added: "+45"
- board text added: "-45"
- board text added: "DANGER 230V"
- board text added: "GND"
- board text added: "L1"
- board text added: "Mains Filter Rectifier 600VA 63V Channel 1"
- board text added: "Mains Filter Rectifier 600VA 63V Channel 2"
- board text added: "N"
- board text added: "V+"
- board text added: "V-"

Commit message: Reviews
Parts:
- added G***: LOGO, TheBrutzlers_Lib:approved_theBrutzler, F.Cu at (252.3, 142.4)
- moved D106 17.0 mm to (144.0, 157.0)
- moved D107 17.0 mm to (127.0, 157.1)
- moved D112 17.0 mm to (265.3, 167.9)
- moved D116 17.0 mm to (282.3, 167.9)
- moved HS102 17.0 mm to (147.5, 162.5)
- moved HS104 17.0 mm to (130.5, 162.5)
- moved HS105 17.0 mm to (279.0, 162.5)
- moved HS107 17.0 mm to (262.0, 162.5)
- moved F103 2.45 mm to (72.5, 146.4)
- moved F102 0.25 mm to (83.3, 146.4)
- moved C107 0.09 mm to (329.8, 123.5)
Routing:
- net Net-(D111-K): track 163.2 -> 252.0 mm
- net Net-(D105-K): track 164.5 -> 244.0 mm
- net Net-(C105-Pad2): track 316.2 -> 254.6 mm
- net Net-(C109-Pad2): track 317.5 -> 260.9 mm
- net GND1: track 34.8 -> 0.00 mm
- net GND2: track 33.7 -> 0.00 mm
- net Net-(D108-K): track 59.9 -> 53.2 mm
- net Net-(D116-K): track 59.6 -> 55.2 mm
- net Net-(D107-K): track 60.0 -> 56.2 mm
- net Net-(D115-K): track 58.7 -> 56.3 mm
- net Net-(J110-Pin_1): track 24.3 -> 25.2 mm
- removed copper zone on B.Cu, net GND1
- removed copper zone on B.Cu, net GND2
- removed copper zone on F.Cu, net Net-(C105-Pad2)
- removed copper zone on F.Cu, net Net-(C109-Pad2)
