File: Hardware/Black_Devil/Softstart.kicad_sch (KiCad schematic)
At the start: 82 parts, among them J101 L1, J102 N, J103 L1_F, J104 N, J105 +45VAC, J106 -45VAC, J107 0V, J108 0V, J109 +63VDC, J110 -63VDC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

Commit message: Major Update
Repo Cleanup
Finished VU Meter PCB
Finalized Softstart PCB
Finalized Channel PCB
Parts:
- C103, C104, C105, C106, C107, C108, C109, C110: value 10.000µ 80V -> 10.000µ 100V
Other:
- note added: "FIN 40.61.8 230V"
- note removed: "FIN 40.52 230V"
Changed lines of the file:
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@@
     (stroke (width 0) (type default))
   )
-  (text "FIN 40.52 230V" (at 190.5 145.415 0)
+  (text "FIN 40.61.8 230V" (at 190.5 145.415 0)
     (effects (font (size 1.27 1.27)) (justify left bottom))
   )
@@
     (effects (font (size 1.27 1.27)) (justify left bottom))
   )
-  (text "FIN 40.52 230V" (at 52.07 144.78 0)
+  (text "FIN 40.61.8 230V" (at 52.07 144.78 0)
     (effects (font (size 1.27 1.27)) (justify left bottom))
   )
@@
       (effects (font (size 1.27 1.27)))
     )
-    (property "Value" "10.000µ 80V" (at 82.55 67.31 90)
+    (property "Value" "10.000µ 100V" (at 82.55 67.31 90)
       (effects (font (size 1.27 1.27)))
     )
@@
       (effects (font (size 1.27 1.27)))
     )
-    (property "Value" "10.000µ 80V" (at 82.55 38.1 90)
+    (property "Value" "10.000µ 100V" (at 82.55 38.1 90)
       (effects (font (size 1.27 1.27)))
     )
@@
       (effects (font (size 1.27 1.27)))
     )
-    (property "Value" "10.000µ 80V" (at 93.345 67.31 90)
+    (property "Value" "10.000µ 100V" (at 93.345 67.31 90)
       (effects (font (size 1.27 1.27)))
     )
@@
       (effects (font (size 1.27 1.27)))
     )
-    (property "Value" "10.000µ 80V" (at 220.345 38.1 90)
+    (property "Value" "10.000µ 100V" (at 220.345 38.1 90)
       (effects (font (size 1.27 1.27)))
     )
@@
       (effects (font (size 1.27 1.27)))
     )
-    (property "Value" "10.000µ 80V" (at 231.14 67.31 90)
+    (property "Value" "10.000µ 100V" (at 231.14 67.31 90)
       (effects (font (size 1.27 1.27)))
     )
@@
       (effects (font (size 1.27 1.27)))
     )
-    (property "Value" "10.000µ 80V" (at 220.345 67.31 90)
+    (property "Value" "10.000µ 100V" (at 220.345 67.31 90)
       (effects (font (size 1.27 1.27)))
     )
@@
       (effects (font (size 1.27 1.27)))
     )
-    (property "Value" "10.000µ 80V" (at 93.345 38.1 90)
+    (property "Value" "10.000µ 100V" (at 93.345 38.1 90)
       (effects (font (size 1.27 1.27)))
     )
@@
       (effects (font (size 1.27 1.27)))
     )
-    (property "Value" "10.000µ 80V" (at 231.14 38.1 90)
+    (property "Value" "10.000µ 100V" (at 231.14 38.1 90)
       (effects (font (size 1.27 1.27)))
     )
@@
     )
   )
+  (sheet_instances
+    (path "/" (page "1"))
+  )
 )
