File: Hardware/Black_Devil/VU-Meter.kicad_pcb (KiCad board)
At the start: 2 copper layers, 62.5 x 80 mm, 155 parts, among them J101 Left, J102 Right, J103 Right, U101 LM2902, U102 LM2902, U103 LM2902, U104 LM2902, U105 LM2902, U106 LM2902, U107 LM2902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

Commit message: Major Update
Repo Cleanup
Finished VU Meter PCB
Finalized Softstart PCB
Finalized Channel PCB
Parts:
- added G***: LOGO, eigene:logo, F.Cu at (132.8, 86.8)
- added REF**: OSHW-Logo2_9.8x8mm_SilkScreen, Symbol:OSHW-Logo2_9.8x8mm_SilkScreen, F.Cu at (132.8, 97.2)
- added REF**: WEEE-Logo_5.6x8mm_SilkScreen, Symbol:WEEE-Logo_5.6x8mm_SilkScreen, F.Cu at (133.0, 114.8)
- added REF**: ESD-Logo_8.9x8mm_SilkScreen, Symbol:ESD-Logo_8.9x8mm_SilkScreen, F.Cu at (132.8, 105.5)
- moved R169 6.00 mm to (118.2, 102.0)
- moved J102 5.08 mm to (79.5, 83.5), turned to -90 degrees
- moved J103 5.08 mm to (135.3, 52.5), turned to 180 degrees
- moved R151 4.50 mm to (124.2, 62.0)
- moved R154 4.50 mm to (119.8, 62.0)
- moved R155 4.50 mm to (119.8, 69.5)
- moved R158 4.50 mm to (124.2, 69.5)
- moved R159 4.50 mm to (124.2, 82.0)
- moved R162 4.50 mm to (119.8, 82.0)
- moved R163 4.50 mm to (119.8, 89.5)
- moved R174 4.50 mm to (124.2, 89.5)
- moved R148 3.00 mm to (119.8, 49.5)
- moved R150 3.00 mm to (122.8, 49.5)
- moved R166 3.00 mm to (122.8, 102.0)
- moved R168 3.00 mm to (119.8, 102.0)
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Connections:
- J102 pad 1: +5VA -> GND
- J102 pad 2: GND -> +5VA
- J103 pad 1: Net-(D119-A) -> GND
- J103 pad 2: GND -> Net-(D119-A)
- R149 pad 2: Net-(U105B--) -> Net-(U105A--)
- R150 pad 2: Net-(U105B--) -> Net-(U105A--)
- R151 pad 2: Net-(U105C--) -> Net-(U105D--)
- R152 pad 2: Net-(U105C--) -> Net-(U105D--)
- R153 pad 2: Net-(U105D--) -> Net-(U105C--)
- R154 pad 2: Net-(U105D--) -> Net-(U105C--)
- R155 pad 2: Net-(U106A--) -> Net-(U106B--)
- R156 pad 2: Net-(U106A--) -> Net-(U106B--)
- R157 pad 2: Net-(U106B--) -> Net-(U106A--)
- R158 pad 2: Net-(U106B--) -> Net-(U106A--)
- R159 pad 2: Net-(U106C--) -> Net-(U106D--)
- R160 pad 2: Net-(U106C--) -> Net-(U106D--)
- R161 pad 2: Net-(U106D--) -> Net-(U106C--)
- R162 pad 2: Net-(U106D--) -> Net-(U106C--)
- R163 pad 2: Net-(U107A--) -> Net-(U107B--)
- R164 pad 2: Net-(U107A--) -> Net-(U107B--)
- R165 pad 2: Net-(U107B--) -> Net-(U107A--)
- R166 pad 2: Net-(U107C--) -> Net-(U107D--)
- R167 pad 2: Net-(U107D--) -> Net-(U107C--)
- R168 pad 2: Net-(U107D--) -> Net-(U107C--)
- R169 pad 2: Net-(U108A--) -> Net-(U108B--)
- R170 pad 2: Net-(U108A--) -> Net-(U108B--)
- R171 pad 2: Net-(U108B--) -> Net-(U108A--)
- R172 pad 2: Net-(U108D--) -> Net-(U108C--)
- R174 pad 1: Net-(U107B--) -> Net-(U107A--)
- R174 pad 2: Net-(U107C--) -> Net-(U107D--)
- R175 pad 1: Net-(U108B--) -> Net-(U108A--)
- R175 pad 2: Net-(U108C--) -> Net-(U108D--)
- R176 pad 1: Net-(U108C--) -> Net-(U108D--)
- R176 pad 2: Net-(U108D--) -> Net-(U108C--)
- U105 pad 1: Net-(D121-A) -> Net-(D122-A)
- U105 pad 14: Net-(D124-A) -> Net-(D123-A)
- U105 pad 2: +5VA -> Net-(U105A--)
- U105 pad 6: Net-(U105B--) -> +5VA
- U105 pad 7: Net-(D122-A) -> Net-(D121-A)
- U105 pad 8: Net-(D123-A) -> Net-(D124-A)
- U106 pad 1: Net-(D125-A) -> Net-(D126-A)
- U106 pad 14: Net-(D128-A) -> Net-(D127-A)
- U106 pad 7: Net-(D126-A) -> Net-(D125-A)
- U106 pad 8: Net-(D127-A) -> Net-(D128-A)
- U107 pad 1: Net-(D129-A) -> Net-(D130-A)
- U107 pad 14: Net-(D132-A) -> Net-(D131-A)
- U107 pad 7: Net-(D130-A) -> Net-(D129-A)
- U107 pad 8: Net-(D131-A) -> Net-(D132-A)
- U108 pad 1: Net-(D133-A) -> Net-(D134-A)
- U108 pad 14: Net-(D136-A) -> Net-(D135-A)
- U108 pad 7: Net-(D134-A) -> Net-(D133-A)
- U108 pad 8: Net-(D135-A) -> Net-(D136-A)
Routing:
- net +5VA: track 108.0 -> 248.9 mm, vias 17 -> 33
- net Net-(D120-K): track 0.00 -> 121.4 mm, vias 0 -> 9
- net Net-(U108A--): track 0.00 -> 20.8 mm
- net Net-(U107D--): track 0.00 -> 18.5 mm
- net Net-(R150-Pad1): track 0.00 -> 16.7 mm
- net GND: track 53.9 -> 70.2 mm, vias 44 -> 56
- net Net-(R158-Pad1): track 0.00 -> 15.9 mm
- net Net-(U108B--): track 0.00 -> 10.8 mm
- net Net-(D131-A): track 0.00 -> 10.6 mm
- net Net-(D135-A): track 0.00 -> 10.6 mm
- net Net-(D134-A): track 0.00 -> 10.6 mm
- net Net-(D130-A): track 0.00 -> 10.6 mm
- net Net-(D127-A): track 0.00 -> 10.6 mm
- net Net-(D126-A): track 0.00 -> 10.6 mm
- net Net-(D123-A): track 0.00 -> 10.5 mm
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Other:
- board text added: "- +"
- board text added: "3 0 -3 -6 -9 -12 -15 -18 -21 -24 -27 -30 -33 -36 -39 -42"
- board text added: "GND +5V"
- board text added: "Stereo VU-Meter 16 LEDs"

Commit message: Finalize all PCBs
Parts:
- RV101, RV102: moved to B.Cu
Connections:
- net Net-(D101-A) renamed /Left
- net Net-(D119-A) renamed /Right
- RV101 pad 1: GND -> Net-(C103-Pad1)
- RV101 pad 3: Net-(C103-Pad1) -> GND
- RV102 pad 1: Net-(C108-Pad1) -> GND
- RV102 pad 3: GND -> Net-(C108-Pad1)
Routing:
- net Net-(D120-K): track 121.4 -> 126.4 mm, vias 9 -> 10
- net GND: track 70.2 -> 66.1 mm, vias 56 -> 54
- net Net-(D102-K): track 119.4 -> 123.1 mm, vias 9 -> 10
- net Net-(C108-Pad1): track 4.24 -> 5.84 mm, vias 0 -> 1
- net Net-(C103-Pad1): track 5.47 -> 6.05 mm, vias 0 -> 1
