File: Hardware/Black_Devil/black_devil.kicad_pcb (KiCad board)
At the start: 2 copper layers, 245 x 60 mm, 120 parts, among them J1 IN, J2 IN_GND, J3 OUT, J4 +63V, J5 -63V, J6 GND, J7 SPK_GND, Q1 2N5551, Q10 MJE350, Q11 MJL3281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

Commit message: Major Update
Repo Cleanup
Finished VU Meter PCB
Finalized Softstart PCB
Finalized Channel PCB
Parts:
- added G***: LOGO, eigene:logo, F.Cu at (43.0, 68.0)
- added REF**: OSHW-Logo2_9.8x8mm_SilkScreen, Symbol:OSHW-Logo2_9.8x8mm_SilkScreen, F.Cu at (43.0, 78.8)
- added REF**: WEEE-Logo_5.6x8mm_SilkScreen, Symbol:WEEE-Logo_5.6x8mm_SilkScreen, F.Cu at (43.0, 97.0)
- added REF**: ESD-Logo_8.9x8mm_SilkScreen, Symbol:ESD-Logo_8.9x8mm_SilkScreen, F.Cu at (43.0, 86.8)

Commit message: Reviews
Parts:
- removed J2: IN_GND, TerminalBlock_MetzConnect:TerminalBlock_MetzConnect_360381_1x01_Horizontal_ScrewM3.0
- J1: value IN -> Input; footprint TerminalBlock_MetzConnect:TerminalBlock_MetzConnect_360381_1x01_Horizontal_ScrewM3.0 -> TerminalBlock:TerminalBlock_bornier-2_P5.08mm
- moved J1 3.88 mm to (37.5, 115.0), turned to 0 degrees
- moved C10 3.50 mm to (40.2, 106.5)
Connections:
- net Net-(J3-Pin_1) renamed /out
Routing:
- net Net-(LED1-K): track 96.9 -> 101.8 mm
- net Net-(Q8-E): track 112.7 -> 114.0 mm
- net Net-(T4-B): track 27.6 -> 28.7 mm

Commit message: Reviews, Gerber Plots and Overview Update
Parts:
- added G***: LOGO, TheBrutzlers_Lib:approved_theBrutzler, F.Cu at (143.8, 65.8)
