File: Hardware/Black_Devil/black_devil.kicad_sch (KiCad schematic)
At the start: 114 parts, among them J1 IN, J2 IN_GND, J3 OUT, J4 +63V, J5 -63V, J6 GND, J7 SPK_GND, Q1 2N5551, Q10 MJE350, Q11 MJL3281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

Commit message: Reviews
Parts:
- removed J1: IN, TerminalBlock_MetzConnect:TerminalBlock_MetzConnect_360381_1x01_Horizontal_ScrewM3.0, symbol Connector_Generic:Conn_01x01
- removed J2: IN_GND, TerminalBlock_MetzConnect:TerminalBlock_MetzConnect_360381_1x01_Horizontal_ScrewM3.0, symbol Connector_Generic:Conn_01x01
- added J1: Input, TerminalBlock:TerminalBlock_bornier-2_P5.08mm, symbol Connector:Screw_Terminal_01x02
Connections:
- net GNDA: now also J1.2 (Pin_2)
- net at C12.1: now also J1.1 (Pin_1)
Changed lines of the file:
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@@
     (stroke (width 0) (type default))
   )
-  (wire (pts (xy 36.83 39.37) (xy 36.83 44.45))
+  (wire (pts (xy 36.83 35.56) (xy 36.83 44.45))
     (stroke (width 0) (type default))
   )
@@
     (stroke (width 0) (type default))
   )
+  (wire (pts (xy 31.115 38.1) (xy 27.94 38.1))
+    (stroke (width 0) (type default))
+  )
   (wire (pts (xy 253.365 121.285) (xy 253.365 128.905))
     (stroke (width 0) (type default))
@@
     (stroke (width 0) (type default))
   )
-  (wire (pts (xy 24.13 118.11) (xy 27.94 118.11))
-    (stroke (width 0) (type default))
-  )
   (wire (pts (xy 372.745 144.145) (xy 372.745 147.955))
     (stroke (width 0) (type default))
@@
     (stroke (width 0) (type default))
   )
+  (wire (pts (xy 31.115 38.1) (xy 31.115 40.64))
+    (stroke (width 0) (type default))
+  )
   (wire (pts (xy 99.06 74.93) (xy 81.28 74.93))
     (stroke (width 0) (type default))
@@
     (stroke (width 0) (type default))
   )
+  (wire (pts (xy 36.83 35.56) (xy 27.94 35.56))
+    (stroke (width 0) (type default))
+  )
   (wire (pts (xy 87.63 131.445) (xy 76.2 131.445))
     (stroke (width 0) (type default))
@@
     (effects (font (size 1.27 1.27)) (justify left bottom))
   )
-  (text "MKS4-100 10µ" (at 16.51 49.53 0)
+  (text "MKS4-100 10µ" (at 38.735 45.085 0)
     (effects (font (size 1.27 1.27)) (justify left bottom))
   )
@@
     )
   )
+  (symbol (lib_id "power:GNDA") (at 31.115 40.64 0) (unit 1)
+    (in_bom yes) (on_board yes) (dnp no) (fields_autoplaced)
+    (property "Reference" "#PWR0101" (at 31.115 46.99 0)
+      (effects (font (size 1.27 1.27)) hide)
+    )
+    (property "Value" "GNDA" (at 31.115 44.7731 0)
+      (effects (font (size 1.27 1.27)))
+    )
+    (property "Footprint" "" (at 31.115 40.64 0)
+      (effects (font (size 1.27 1.27)) hide)
+    )
+    (property "Datasheet" "" (at 31.115 40.64 0)
+      (effects (font (size 1.27 1.27)) hide)
+    )
+    (pin "1")
+    (instances
+      (project "black_devil"
+        (path "/07eb527d-7924-4a90-98a2-747aa2a8ca8b"
+          (reference "#PWR0101") (unit 1)
+        )
+      )
+      (project "Overview_Schematic"
+        (path "/c7b1811f-24fd-4e13-a38a-b587cd9cacbf/007584f1-313f-4eff-a9e4-7f530c98a9bb"
+          (reference "#PWR01") (unit 1)
+        )
+        (path "/c7b1811f-24fd-4e13-a38a-b587cd9cacbf/ae5c1915-c4d9-4eb1-92e9-03a1facb5d93"
+          (reference "#PWR015") (unit 1)
+        )
+      )
+    )
+  )
   (symbol (lib_id "Device:R") (at 73.66 56.515 0) (unit 1)
     (in_bom yes) (on_board yes) (dnp no) (fields_autoplaced)
@@
     )
   )
-  (symbol (lib_id "Connector_Generic:Conn_01x01") (at 19.05 118.11 180) (unit 1)
-    (in_bom yes) (on_board yes) (dnp no) (fields_autoplaced)
-    (property "Reference" "J2" (at 19.05 112.6957 0)
-      (effects (font (size 1.27 1.27)))
-    )
-    (property "Value" "IN_GND" (at 19.05 115.1199 0)
-      (effects (font (size 1.27 1.27)))
-    )
-    (property "Footprint" "TerminalBlock_MetzConnect:TerminalBlock_MetzConnect_360381_1x01_Horizontal_ScrewM3.0" (at 19.05 118.11 0)
-      (effects (font (size 1.27 1.27)) hide)
-    )
-    (property "Datasheet" "~" (at 19.05 118.11 0)
-      (effects (font (size 1.27 1.27)) hide)
-    )
-    (pin "1")
-    (instances
-      (project "black_devil"
-        (path "/07eb527d-7924-4a90-98a2-747aa2a8ca8b"
-          (reference "J2") (unit 1)
-        )
-      )
-      (project "Overview_Schematic"
-        (path "/c7b1811f-24fd-4e13-a38a-b587cd9cacbf/007584f1-313f-4eff-a9e4-7f530c98a9bb"
-          (reference "J2") (unit 1)
-        )
-        (path "/c7b1811f-24fd-4e13-a38a-b587cd9cacbf/ae5c1915-c4d9-4eb1-92e9-03a1facb5d93"
-          (reference "J11") (unit 1)
-        )
-      )
-    )
-  )
   (symbol (lib_id "Device:R") (at 274.955 112.395 0) (mirror x) (unit 1)
     (in_bom yes) (on_board yes) (dnp no)
@@
     )
   )
+  (symbol (lib_id "Connector:Screw_Terminal_01x02") (at 22.86 35.56 0) (mirror y) (unit 1)
+    (in_bom yes) (on_board yes) (dnp no)
+    (property "Reference" "J1" (at 20.828 35.6179 0)
+      (effects (font (size 1.27 1.27)) (justify left))
+    )
+    (property "Value" "Input" (at 20.828 38.0421 0)
+      (effects (font (size 1.27 1.27)) (justify left))
+    )
+    (property "Footprint" "TerminalBlock:TerminalBlock_bornier-2_P5.08mm" (at 22.86 35.56 0)
+      (effects (font (size 1.27 1.27)) hide)
+    )
+    (property "Datasheet" "~" (at 22.86 35.56 0)
+      (effects (font (size 1.27 1.27)) hide)
+    )
+    (pin "1")
+    (pin "2")
+    (instances
+      (project "black_devil"
+        (path "/07eb527d-7924-4a90-98a2-747aa2a8ca8b"
+          (reference "J1") (unit 1)
+        )
+      )
+      (project "digital"
+        (path "/6cfa901a-81f3-4fe2-a026-5f0c8f3321de"
+          (reference "J111") (unit 1)
+        )
+      )
+      (project "Overview_Schematic"
+        (path "/c7b1811f-24fd-4e13-a38a-b587cd9cacbf/60e79a5f-d737-4a43-902b-ccd082ad4ee1"
+          (reference "J508") (unit 1)
+        )
+      )
+    )
+  )
   (symbol (lib_id "Device:LED") (at 76.2 139.7 90) (unit 1)
     (in_bom yes) (on_board yes) (dnp no) (fields_autoplaced)
@@
         )
       )
-    )
-  )
-  (symbol (lib_id "Connector_Generic:Conn_01x01") (at 36.83 34.29 90) (unit 1)
-    (in_bom yes) (on_board yes) (dnp no) (fields_autoplaced)
-    (property "Reference" "J1" (at 38.862 33.0779 90)
-      (effects (font (size 1.27 1.27)) (justify right))
-    )
-    (property "Value" "IN" (at 38.862 35.5021 90)
-      (effects (font (size 1.27 1.27)) (justify right))
-    )
-    (property "Footprint" "TerminalBlock_MetzConnect:TerminalBlock_MetzConnect_360381_1x01_Horizontal_ScrewM3.0" (at 36.83 34.29 0)
-      (effects (font (size 1.27 1.27)) hide)
-    )
-    (property "Datasheet" "~" (at 36.83 34.29 0)
-      (effects (font (size 1.27 1.27)) hide)
-    )
-    (pin "1")
-    (instances
-      (project "black_devil"
-        (path "/07eb527d-7924-4a90-98a2-747aa2a8ca8b"
-          (reference "J1") (unit 1)
-        )
-      )
-      (project "Overview_Schematic"
-        (path "/c7b1811f-24fd-4e13-a38a-b587cd9cacbf/007584f1-313f-4eff-a9e4-7f530c98a9bb"
-          (reference "J1") (unit 1)
-        )
-        (path "/c7b1811f-24fd-4e13-a38a-b587cd9cacbf/ae5c1915-c4d9-4eb1-92e9-03a1facb5d93"
-          (reference "J8") (unit 1)
-        )
-      )
