File: Hardware/Black_Devil/digital.kicad_sch (KiCad schematic)
At the start: 62 parts, among them J5 L1, J5 N, J503 Left, J504 Right, J505 Klinke_Right, J506 Klinke_Links, J507 Cinch_Right, J508 Cinch_Left, J509 OLED, K501 G6K-2, K502 G6K-2, K503 G6K-2, Q501 BSS138, Q502 BSS138, Q503 BSS138, T501 4815-2, U501 L7805, U502 L7805, U503 AP1117-33, U505 ATmega328P-A, Y501 16MHz

Commit message: Major Update
Repo Cleanup
Finished VU Meter PCB
Finalized Softstart PCB
Finalized Channel PCB
Parts:
- removed C513, C516: 1µ, symbol Device:C
- removed C514, C515: 100n, symbol Device:C
- removed U503: AP1117-33, Package_TO_SOT_SMD:SOT-223-3_TabPin2, symbol Regulator_Linear:AP1117-33
- T501: value 4815-2 -> UI 39/10,2 209
Other:
- note added: "9V 777mA"
- note removed: "7,5V 666mA"

Commit message: Finalize all PCBs
Parts:
- removed R509, R510: 4k7, symbol Device:R
- removed T501: UI 39/10,2 209, symbol Device:Transformer_1P_2S
- added C114, C119: 1µ, Capacitor_SMD:C_0805_2012Metric, symbol Device:C
- added C116, C118, C120: 100n, Capacitor_SMD:C_0805_2012Metric, symbol Device:C
- added J103: UART, Connector_JST:JST_XH_B3B-XH-A_1x03_P2.50mm_Vertical, symbol Connector_Generic:Conn_01x03
- added J105: Encoder, Connector_JST:JST_XH_B5B-XH-A_1x05_P2.50mm_Vertical, symbol Connector_Generic:Conn_01x05
- added J106: Up2Stream, TerminalBlock:TerminalBlock_bornier-2_P5.08mm, symbol Connector:Screw_Terminal_01x02
- added J107: ICSP, Connector_PinHeader_2.54mm:PinHeader_2x03_P2.54mm_Vertical, symbol Connector_Generic:Conn_02x03_Odd_Even
- added J114: VU-Meter, TerminalBlock:TerminalBlock_bornier-2_P5.08mm, symbol Connector:Screw_Terminal_01x02
- added J115: Up2Stream, TerminalBlock:TerminalBlock_bornier-4_P5.08mm, symbol Connector:Screw_Terminal_01x04
- added Q101, Q102, Q103, Q104: BSS138, Package_TO_SOT_SMD:SOT-23, symbol Transistor_FET:BSS138
- added R101, R102, R103, R104, R105, R106, R107, R108: 4k7, Resistor_SMD:R_0805_2012Metric, symbol Device:R
- added R111, R112, R113: 10k, Resistor_SMD:R_0805_2012Metric, symbol Device:R
- added SW101: RotaryEncoder_Switch, Rotary_Encoder:RotaryEncoder_Bourns_Horizontal_PEC09-2xxxF-Sxxxx, symbol Device:RotaryEncoder_Switch
- added TP101: PD2, TestPoint:TestPoint_Loop_D2.50mm_Drill1.0mm, symbol Connector:TestPoint
- added TP102: PD3, TestPoint:TestPoint_Loop_D2.50mm_Drill1.0mm, symbol Connector:TestPoint
- added TP103: PD4, TestPoint:TestPoint_Loop_D2.50mm_Drill1.0mm, symbol Connector:TestPoint
- added TP104: 9V, TestPoint:TestPoint_Loop_D2.50mm_Drill1.0mm, symbol Connector:TestPoint
- added TP105: GND, TestPoint:TestPoint_Loop_D2.50mm_Drill1.0mm, symbol Connector:TestPoint
- added TR101: UI 39/10,2 209, eigene:BLOCK 14VA, symbol Transformer:TRANSF6
- added U104: AP1117-33, Package_TO_SOT_SMD:SOT-223-3_TabPin2, symbol Regulator_Linear:AP1117-33
- C101: renamed from C501; footprint (none) -> Capacitor_SMD:C_0805_2012Metric
- C102: renamed from C502; footprint (none) -> Capacitor_SMD:C_0805_2012Metric
- C103: renamed from C503; footprint (none) -> Capacitor_SMD:C_0805_2012Metric
- C104: renamed from C504; footprint (none) -> Capacitor_SMD:C_0805_2012Metric
- C105: renamed from C519; footprint (none) -> Capacitor_SMD:C_0805_2012Metric
- C106: renamed from C517; footprint (none) -> Capacitor_SMD:C_0805_2012Metric
- C107: renamed from C518; footprint (none) -> Capacitor_SMD:C_0805_2012Metric
- C108: renamed from C505; footprint (none) -> Capacitor_THT:CP_Radial_D10.0mm_P5.00mm
- C109: renamed from C506; footprint (none) -> Capacitor_THT:CP_Radial_D10.0mm_P5.00mm
- C110: renamed from C507; footprint (none) -> Capacitor_THT:CP_Radial_D10.0mm_P5.00mm
- C111: renamed from C509; footprint (none) -> Capacitor_SMD:C_0805_2012Metric
- C112: renamed from C510; footprint (none) -> Capacitor_SMD:C_0805_2012Metric
- C113: renamed from C508; footprint (none) -> Capacitor_THT:CP_Radial_D10.0mm_P5.00mm
- C115: renamed from C511; footprint (none) -> Capacitor_SMD:C_0805_2012Metric
- C117: renamed from C512; footprint (none) -> Capacitor_SMD:C_0805_2012Metric
- HS101: renamed from HS501; footprint (none) -> eigene:V 4330N
- HS102: renamed from HS502; footprint (none) -> eigene:V 4330N
- J104: renamed from J509; footprint (none) -> Connector_JST:JST_XH_B4B-XH-A_1x04_P2.50mm_Vertical
- J108: renamed from J505; footprint (none) -> TerminalBlock:TerminalBlock_bornier-2_P5.08mm
- J109: renamed from J506; footprint (none) -> TerminalBlock:TerminalBlock_bornier-2_P5.08mm
- J110: renamed from J507; footprint (none) -> TerminalBlock:TerminalBlock_bornier-2_P5.08mm
- J111: renamed from J508; footprint (none) -> TerminalBlock:TerminalBlock_bornier-2_P5.08mm
- J112: renamed from J503; footprint (none) -> TerminalBlock:TerminalBlock_bornier-2_P5.08mm
- J113: renamed from J504; footprint (none) -> TerminalBlock:TerminalBlock_bornier-2_P5.08mm
- K101: renamed from K501; footprint (none) -> Relay_SMD:Relay_DPDT_Omron_G6K-2F
- K102: renamed from K502; footprint (none) -> Relay_SMD:Relay_DPDT_Omron_G6K-2F
- K103: renamed from K503; footprint (none) -> Relay_SMD:Relay_DPDT_Omron_G6K-2F
- R109: renamed from R501; footprint (none) -> Resistor_SMD:R_0805_2012Metric
- R110: renamed from R502; footprint (none) -> Resistor_SMD:R_0805_2012Metric
- R114: renamed from R507; footprint (none) -> Resistor_SMD:R_0805_2012Metric
- R115: renamed from R505; footprint (none) -> Resistor_SMD:R_0805_2012Metric
- R116: renamed from R503; footprint (none) -> Resistor_SMD:R_0805_2012Metric
- R117: renamed from R508; footprint (none) -> Resistor_SMD:R_0805_2012Metric
- R118: renamed from R506; footprint (none) -> Resistor_SMD:R_0805_2012Metric
- R119: renamed from R504; footprint (none) -> Resistor_SMD:R_0805_2012Metric
- R120: renamed from R511; footprint (none) -> Resistor_SMD:R_0805_2012Metric
- R121: renamed from R512; footprint (none) -> Resistor_SMD:R_0805_2012Metric
- U102: renamed from U501; footprint (none) -> Package_TO_SOT_THT:TO-220-3_Vertical
- U103: renamed from U502; footprint (none) -> Package_TO_SOT_THT:TO-220-3_Vertical
- Y101: renamed from Y501; footprint (none) -> Crystal:Crystal_SMD_HC49-SD
- renumbered D501 to D101, D503 to D102, D502 to D103, D504 to D104, D507 to D105, D506 to D106, D505 to D107, Q503 to Q105, Q502 to Q106, Q501 to Q107, U505 to U101
Connections:
- net +5V: now also J106.1 (Pin_1)
- net +5VA: now also C114.1, C116.1, C120.1, J105.2 (Pin_2), J107.2 (Pin_2), J114.1 (Pin_1), Q101.1 (G), Q102.1 (G), Q103.1 (G), Q104.1 (G), R101.1, R102.1, R103.1, R104.1, R111.1, R112.1, R113.1, U104.3 (VI); no longer J104.1 (Pin_1)
- net GND: now also C114.2, C116.2, C118.2, C119.2, C120.2, J103.1 (Pin_1), J105.1 (Pin_1), J106.2 (Pin_2), J107.6 (Pin_6), J114.2 (Pin_2), J115.2 (Pin_2), J115.4 (Pin_4), SW101.C, SW101.S2, TP105.1, U104.1 (GND)
- net N: now also TR101.4
- net RxD: now also Q101.2 (S), R101.2
- net SCL: now also Q103.2 (S), R103.2; no longer J104.3 (Pin_3)
- net SDA: now also Q104.2 (S), R104.2; no longer J104.4 (Pin_4)
- net TxD: now also Q102.2 (S), R102.2
- net at D101.2 (A), D102.1 (K): now also TR101.6, TR101.8
- net at D103.2 (A), D104.1 (K): now also TR101.5, TR101.7
- net RST: now reaches C105.1, R110.2, U101.29 (~{RESET}/PC6)
- net RST: now also J107.5 (Pin_5)
- net at F101.2: now also TR101.1
- net at U101.1 (PD3): now also TP102.1
- net at U101.10 (PD6): now also J105.4 (Pin_4), R111.2, SW101.A
- net at U101.11 (PD7): now also J105.5 (Pin_5), R112.2, SW101.B
- net MISO: now reaches U101.15 (PB3)
- net MISO: now also J107.1 (Pin_1)
- net MOSI: now reaches U101.16 (PB4)
- net MOSI: now also J107.4 (Pin_4)
- net SCK: now reaches U101.17 (PB5)
- net SCK: now also J107.3 (Pin_3)
- net at U101.2 (PD4): now also TP103.1
- net at U101.32 (PD2): now also TP101.1
- net at U101.9 (PD5): now also J105.3 (Pin_3), R113.2, SW101.S1
- net +9V renamed +12V
- net +12V: now also TP104.1
- net Up2Stream_Left: no longer names the net of K103.5
- net Up2Stream_Left: now also J115.3 (Pin_3)
- net Up2Stream_Right: no longer names the net of K103.4
- net Up2Stream_Right: now also J115.1 (Pin_1)
- new net: J103.2 (Pin_2), Q101.3 (D), R105.2
- new net: J104.4 (Pin_4), Q104.3 (D), R108.2
- new net: J104.3 (Pin_3), Q103.3 (D), R107.2
- new net: J103.3 (Pin_3), Q102.3 (D), R106.2
- new net: TR101.2, TR101.3
- new net +3V3: C118.1, C119.1, J104.1 (Pin_1), R105.1, R106.1, R107.1, R108.1, U104.2 (VO)
- no-connect marks 6 -> 12
Other:
- moved on the sheet: C101, C102, C103, C104, C105, C106, C107, C108, C109, C110, C111, C112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

Commit message: Reviews
Parts:
- removed J103: UART, Connector_JST:JST_XH_B3B-XH-A_1x03_P2.50mm_Vertical, symbol Connector_Generic:Conn_01x03
- removed Q101, Q102: BSS138, Package_TO_SOT_SMD:SOT-23, symbol Transistor_FET:BSS138
- removed R105, R106: 4k7, Resistor_SMD:R_0805_2012Metric, symbol Device:R
- removed TP104: 9V, TestPoint:TestPoint_Loop_D2.50mm_Drill1.0mm, symbol Connector:TestPoint
- removed TP105: GND, TestPoint:TestPoint_Loop_D2.50mm_Drill1.0mm, symbol Connector:TestPoint
- added C121, C122, C123, C124: 470µ, Capacitor_THT:CP_Radial_D10.0mm_P5.00mm, symbol Device:C_Polarized
- added C125, C126: 1µ, Capacitor_SMD:C_0805_2012Metric, symbol Device:C
- added C127, C128: 100n, Capacitor_SMD:C_0805_2012Metric, symbol Device:C
- added D108, D109, D110, D111: 1N4004, Diode_THT:D_DO-41_SOD81_P10.16mm_Horizontal, symbol Diode:1N4004
- added J103: OLED, Connector_JST:JST_XH_B4B-XH-A_1x04_P2.50mm_Vertical, symbol Connector_Generic:Conn_01x04
- added TH101, TH102: Thermistor_NTC, Connector_PinHeader_2.54mm:PinHeader_1x02_P2.54mm_Vertical, symbol Device:Thermistor_NTC
- added U105: ADuM1201AR, Package_SO:SOIC-8_3.9x4.9mm_P1.27mm, symbol Isolator:ADuM1201AR
Connections:
- net +12V: now also C121.1, C122.1, C123.1, C124.1, D108.1 (K), D110.1 (K); no longer C101.1, C102.1, C108.1, C109.1, C110.1, C113.1, D101.1 (K), D103.1 (K), U102.1 (IN)
- net +3V3: now also Q103.1 (G), Q104.1 (G)
- net +5V: now also C114.1, C115.1, C116.1, C117.1, C120.1, D105.1 (K), D106.1 (K), D107.1 (K), J105.2 (Pin_2), J107.2 (Pin_2), J114.1 (Pin_1), K101.1, K102.1, K103.1, R101.1, R102.2, R103.1, R104.1, R110.1, R111.1, R112.1, R113.1, U101.18 (AVCC), U101.20 (AREF), U101.4 (VCC), U101.6 (VCC), U103.3 (OUT), U104.3 (VI), C127.1, U105.1 (VDD1); no longer C103.1, C104.1, J106.1 (Pin_1), U102.3 (OUT)
- net +5VA: now also C103.1, C104.1, J106.1 (Pin_1), U102.3 (OUT); no longer C114.1, C115.1, C116.1, C117.1, C120.1, D105.1 (K), D106.1 (K), D107.1 (K), J105.2 (Pin_2), J107.2 (Pin_2), J114.1 (Pin_1), K101.1, K102.1, K103.1, Q103.1 (G), Q104.1 (G), R101.1, R102.1, R103.1, R104.1, R110.1, R111.1, R112.1, R113.1, U101.18 (AVCC), U101.20 (AREF), U101.4 (VCC), U101.6 (VCC), U103.3 (OUT), U104.3 (VI)
- net GND: now also C121.2, C122.2, C123.2, C124.2, C125.1, C126.2, C127.2, D109.2 (A), D111.2 (A), TH101.2, TH102.2, U105.4 (GND1); no longer C101.2, C102.2, C103.2, C104.2, C108.2, C109.2, C110.2, C113.2, D102.2 (A), D104.2 (A), J106.2 (Pin_2), J108.2 (Pin_2), J109.2 (Pin_2), J110.2 (Pin_2), J111.2 (Pin_2), J112.2 (Pin_2), J113.2 (Pin_2), J115.2 (Pin_2), J115.4 (Pin_4), R120.2, R121.2, U102.2 (GND)
- net RxD: now also U105.2 (VOA); no longer R101.2
- net SCL: now also Q103.3 (D); no longer Q103.2 (S)
- net SDA: now also Q104.3 (D); no longer Q104.2 (S)
- net TxD: now also U105.3 (VIB); no longer R102.2
- net at D101.2 (A), D102.1 (K), TR101.8: no longer TR101.6
- net at J104.4 (Pin_4), R108.2: now also Q104.2 (S); no longer Q104.3 (D)
- net at D103.2 (A), D104.1 (K), TR101.7: no longer TR101.5
- net at J104.3 (Pin_3), R107.2: now also Q103.2 (S); no longer Q103.3 (D)
- net NTC1: now reaches U101.23 (PC0)
- net NTC1: now also R101.2, C125.2, TH101.1
- net NTC2: now reaches U101.24 (PC1)
- net NTC2: now also R102.1, C126.1, TH102.1
- new net: D108.2 (A), D109.1 (K), TR101.6
- new net: C128.1, J103.1 (Pin_1), U105.8 (VDD2)
- new net: J103.2 (Pin_2), U105.7 (VIA)
- new net: J103.3 (Pin_3), U105.6 (VOB)
- new net: D110.2 (A), D111.1 (K), TR101.5
- new net +12VA: C101.1, C102.1, C108.1, C109.1, C110.1, C113.1, D101.1 (K), D103.1 (K), U102.1 (IN)
- new net GND1: C101.2, C102.2, C103.2, C104.2, C108.2, C109.2, C110.2, C113.2, C128.2, D102.2 (A), D104.2 (A), J103.4 (Pin_4), J106.2 (Pin_2), U102.2 (GND), U105.5 (GND2)
- new net Sig_GND: J108.2 (Pin_2), J109.2 (Pin_2), J110.2 (Pin_2), J111.2 (Pin_2), J112.2 (Pin_2), J113.2 (Pin_2), J115.2 (Pin_2), J115.4 (Pin_4), R120.2, R121.2
- no-connect marks 12 -> 10
Other:
- note added: "3V3 TxD RxD GND"
- note added: "9V 1333mA"
- note removed: "9V 777mA"
- moved on the sheet: C101, C102, C103, C104, C105, C106, C107, C108, C109, C110, C111, C112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

Commit message: Reviews, Gerber Plots and Overview Update
Parts:
- added TP104, TP105: TestPoint, TestPoint:TestPoint_Loop_D2.50mm_Drill1.0mm, symbol Connector:TestPoint
Connections:
- net +5V: now also TP105.1
- net GND: now also TP104.1
Changed lines of the file:
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@@
     (stroke (width 0) (type default))
   )
+  (wire (pts (xy 69.85 164.465) (xy 69.85 162.56))
+    (stroke (width 0) (type default))
+  )
   (wire (pts (xy 282.575 52.07) (xy 282.575 53.975))
     (stroke (width 0) (type default))
@@
     (stroke (width 0) (type default))
   )
+  (wire (pts (xy 69.85 149.86) (xy 69.85 151.765))
+    (stroke (width 0) (type default))
+  )
   (wire (pts (xy 371.475 159.385) (xy 371.475 161.29))
     (stroke (width 0) (type default))
@@
         )
       )
+      (project "Overview_Schematic"
+        (path "/c7b1811f-24fd-4e13-a38a-b587cd9cacbf/60e79a5f-d737-4a43-902b-ccd082ad4ee1"
+          (reference "J115") (unit 1)
+        )
+      )
     )
   )
@@
         )
       )
+      (project "Overview_Schematic"
+        (path "/c7b1811f-24fd-4e13-a38a-b587cd9cacbf/60e79a5f-d737-4a43-902b-ccd082ad4ee1"
+          (reference "#FLG0104") (unit 1)
+        )
+      )
     )
   )
@@
         )
       )
+      (project "Overview_Schematic"
+        (path "/c7b1811f-24fd-4e13-a38a-b587cd9cacbf/60e79a5f-d737-4a43-902b-ccd082ad4ee1"
+          (reference "#PWR0146") (unit 1)
+        )
+      )
     )
   )
@@
         )
       )
+      (project "Overview_Schematic"
+        (path "/c7b1811f-24fd-4e13-a38a-b587cd9cacbf/60e79a5f-d737-4a43-902b-ccd082ad4ee1"
+          (reference "#PWR0105") (unit 1)
+        )
+      )
     )
   )
@@
         )
       )
+      (project "Overview_Schematic"
+        (path "/c7b1811f-24fd-4e13-a38a-b587cd9cacbf/60e79a5f-d737-4a43-902b-ccd082ad4ee1"
+          (reference "#PWR0109") (unit 1)
+        )
+      )
     )
   )
@@
         )
       )
+      (project "Overview_Schematic"
+        (path "/c7b1811f-24fd-4e13-a38a-b587cd9cacbf/60e79a5f-d737-4a43-902b-ccd082ad4ee1"
+          (reference "TH102") (unit 1)
+        )
+      )
     )
   )
@@
         )
       )
+      (project "Overview_Schematic"
+        (path "/c7b1811f-24fd-4e13-a38a-b587cd9cacbf/60e79a5f-d737-4a43-902b-ccd082ad4ee1"
+          (reference "#FLG0101") (unit 1)
+        )
+      )
     )
   )
@@
         )
       )
+      (project "Overview_Schematic"
+        (path "/c7b1811f-24fd-4e13-a38a-b587cd9cacbf/60e79a5f-d737-4a43-902b-ccd082ad4ee1"
+          (reference "#PWR0126") (unit 1)
+        )
+      )
     )
   )
@@
         )
       )
+      (project "Overview_Schematic"
+        (path "/c7b1811f-24fd-4e13-a38a-b587cd9cacbf/60e79a5f-d737-4a43-902b-ccd082ad4ee1"
+          (reference "#PWR0101") (unit 1)
+        )
+      )
     )
   )
@@
         )
       )
+      (project "Overview_Schematic"
+        (path "/c7b1811f-24fd-4e13-a38a-b587cd9cacbf/60e79a5f-d737-4a43-902b-ccd082ad4ee1"
+          (reference "#FLG0102") (unit 1)
+        )
+      )
     )
   )
@@
         )
       )
+      (project "Overview_Schematic"
+        (path "/c7b1811f-24fd-4e13-a38a-b587cd9cacbf/60e79a5f-d737-4a43-902b-ccd082ad4ee1"
+          (reference "#PWR0148") (unit 1)
+        )
+      )
     )
   )
@@
         )
       )
+      (project "Overview_Schematic"
+        (path "/c7b1811f-24fd-4e13-a38a-b587cd9cacbf/60e79a5f-d737-4a43-902b-ccd082ad4ee1"
+          (reference "#PWR0127") (unit 1)
+        )
+      )
     )
   )
@@
         )
       )
+      (project "Overview_Schematic"
+        (path "/c7b1811f-24fd-4e13-a38a-b587cd9cacbf/60e79a5f-d737-4a43-902b-ccd082ad4ee1"
+          (reference "#FLG0103") (unit 1)
+        )
+      )
+    )
+  )
+  (symbol (lib_id "Connector:TestPoint") (at 69.85 149.86 0) (unit 1)
+    (in_bom yes) (on_board yes) (dnp no) (fields_autoplaced)
+    (property "Reference" "TP105" (at 71.247 145.3459 0)
+      (effects (font (size 1.27 1.27)) (justify left))
+    )
+    (property "Value" "TestPoint" (at 71.247 147.7701 0)
+      (effects (font (size 1.27 1.27)) (justify left))
+    )
+    (property "Footprint" "TestPoint:TestPoint_Loop_D2.50mm_Drill1.0mm" (at 74.93 149.86 0)
+      (effects (font (size 1.27 1.27)) hide)
+    )
+    (property "Datasheet" "~" (at 74.93 149.86 0)
+      (effects (font (size 1.27 1.27)) hide)
+    )
+    (pin "1")
+    (instances
+      (project "digital"
+        (path "/6cfa901a-81f3-4fe2-a026-5f0c8f3321de"
+          (reference "TP105") (unit 1)
+        )
+      )
+      (project "Overview_Schematic"
+        (path "/c7b1811f-24fd-4e13-a38a-b587cd9cacbf/60e79a5f-d737-4a43-902b-ccd082ad4ee1"
+          (reference "TP105") (unit 1)
+        )
+      )
     )
   )
@@
         )
       )
+      (project "Overview_Schematic"
+        (path "/c7b1811f-24fd-4e13-a38a-b587cd9cacbf/60e79a5f-d737-4a43-902b-ccd082ad4ee1"
+          (reference "TR101") (unit 1)
+        )
+      )
+    )
+  )
+  (symbol (lib_id "Connector:TestPoint") (at 69.85 164.465 180) (unit 1)
+    (in_bom yes) (on_board yes) (dnp no) (fields_autoplaced)
+    (property "Reference" "TP104" (at 71.247 166.5549 0)
+      (effects (font (size 1.27 1.27)) (justify right))
+    )
+    (property "Value" "TestPoint" (at 71.247 168.9791 0)
+      (effects (font (size 1.27 1.27)) (justify right))
+    )
+    (property "Footprint" "TestPoint:TestPoint_Loop_D2.50mm_Drill1.0mm" (at 64.77 164.465 0)
+      (effects (font (size 1.27 1.27)) hide)
+    )
+    (property "Datasheet" "~" (at 64.77 164.465 0)
+      (effects (font (size 1.27 1.27)) hide)
+    )
+    (pin "1")
+    (instances
+      (project "digital"
+        (path "/6cfa901a-81f3-4fe2-a026-5f0c8f3321de"
+          (reference "TP104") (unit 1)
+        )
+      )
+      (project "Overview_Schematic"
+        (path "/c7b1811f-24fd-4e13-a38a-b587cd9cacbf/60e79a5f-d737-4a43-902b-ccd082ad4ee1"
+          (reference "TP104") (unit 1)
+        )
+      )
     )
   )
@@
         )
       )
+      (project "Overview_Schematic"
+        (path "/c7b1811f-24fd-4e13-a38a-b587cd9cacbf/60e79a5f-d737-4a43-902b-ccd082ad4ee1"
+          (reference "U105") (unit 1)
+        )
+      )
     )
   )
@@
         )
       )
+      (project "Overview_Schematic"
+        (path "/c7b1811f-24fd-4e13-a38a-b587cd9cacbf/60e79a5f-d737-4a43-902b-ccd082ad4ee1"
+          (reference "TH101") (unit 1)
+        )
+      )
     )
   )
@@
           (reference "#PWR0128") (unit 1)
         )
+      )
+      (project "Overview_Schematic"
+        (path "/c7b1811f-24fd-4e13-a38a-b587cd9cacbf/60e79a5f-d737-4a43-902b-ccd082ad4ee1"
+          (reference "#PWR0128") (unit 1)
+        )
