File: Hardware/Black_Devil/Overview_Schematic.kicad_sch (KiCad schematic)
At the start: 11 parts, among them J15 Conn_01x03_Socket, J16 Klinke, J17 4mm, J18 Speakon, J19 Speakon, J20 4mm, J21 Klinke, T7 2x 45V 600VA, T8 2x 45V 600VA

Commit message: Major Update
Repo Cleanup
Finished VU Meter PCB
Finalized Softstart PCB
Finalized Channel PCB
Other:
- sheet VU_Meter ports: added 5V, GND, Left, Right; removed none
Changed lines of the file:
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@@
   (junction (at 255.27 87.63) (diameter 0) (color 0 0 0 0)
   )
+  (junction (at 241.3 143.51) (diameter 0) (color 0 0 0 0)
+  )
   (junction (at 173.99 92.71) (diameter 0) (color 0 0 0 0)
   )
   (junction (at 261.62 99.695) (diameter 0) (color 0 0 0 0)
   )
+  (junction (at 241.3 92.71) (diameter 0) (color 0 0 0 0)
+  )
   (junction (at 51.435 106.68) (diameter 0) (color 0 0 0 0)
   )
@@
     (stroke (width 0) (type default))
   )
-  (wire (pts (xy 243.205 150.495) (xy 255.27 150.495))
+  (wire (pts (xy 241.3 150.495) (xy 255.27 150.495))
     (stroke (width 0) (type default))
   )
@@
     (stroke (width 0) (type default))
   )
+  (wire (pts (xy 163.83 32.385) (xy 198.755 32.385))
+    (stroke (width 0) (type default))
+  )
   (wire (pts (xy 99.06 98.425) (xy 90.17 98.425))
     (stroke (width 0) (type default))
@@
     (stroke (width 0) (type default))
   )
+  (wire (pts (xy 198.755 62.23) (xy 193.675 62.23))
+    (stroke (width 0) (type default))
+  )
   (wire (pts (xy 171.45 137.795) (xy 171.45 149.225))
     (stroke (width 0) (type default))
@@
     (stroke (width 0) (type default))
   )
-  (wire (pts (xy 234.95 92.71) (xy 252.095 92.71))
+  (wire (pts (xy 234.95 92.71) (xy 241.3 92.71))
+    (stroke (width 0) (type default))
+  )
+  (wire (pts (xy 198.755 64.135) (xy 195.58 64.135))
     (stroke (width 0) (type default))
   )
@@
     (stroke (width 0) (type default))
   )
+  (wire (pts (xy 193.675 135.89) (xy 241.3 135.89))
+    (stroke (width 0) (type default))
+  )
   (wire (pts (xy 49.53 104.14) (xy 55.88 104.14))
     (stroke (width 0) (type default))
@@
     (stroke (width 0) (type default))
   )
-  (wire (pts (xy 234.95 94.615) (xy 243.205 94.615))
+  (wire (pts (xy 234.95 94.615) (xy 241.3 94.615))
     (stroke (width 0) (type default))
   )
@@
     (stroke (width 0) (type default))
   )
+  (wire (pts (xy 241.3 135.89) (xy 241.3 143.51))
+    (stroke (width 0) (type default))
+  )
   (wire (pts (xy 90.17 107.315) (xy 185.42 107.315))
     (stroke (width 0) (type default))
   )
+  (wire (pts (xy 163.83 34.29) (xy 198.755 34.29))
+    (stroke (width 0) (type default))
+  )
+  (wire (pts (xy 241.3 143.51) (xy 252.095 143.51))
+    (stroke (width 0) (type default))
+  )
   (wire (pts (xy 90.17 101.6) (xy 125.095 101.6))
     (stroke (width 0) (type default))
   )
+  (wire (pts (xy 195.58 64.135) (xy 195.58 84.455))
+    (stroke (width 0) (type default))
+  )
   (wire (pts (xy 163.83 40.005) (xy 173.99 40.005))
     (stroke (width 0) (type default))
@@
     (stroke (width 0) (type default))
   )
+  (wire (pts (xy 241.3 84.455) (xy 241.3 92.71))
+    (stroke (width 0) (type default))
+  )
   (wire (pts (xy 185.42 98.425) (xy 207.645 98.425))
     (stroke (width 0) (type default))
@@
     (stroke (width 0) (type default))
   )
+  (wire (pts (xy 195.58 84.455) (xy 241.3 84.455))
+    (stroke (width 0) (type default))
+  )
   (wire (pts (xy 32.385 110.49) (xy 32.385 109.22))
     (stroke (width 0) (type default))
@@
     (stroke (width 0) (type default))
   )
-  (wire (pts (xy 243.205 99.695) (xy 255.27 99.695))
-    (stroke (width 0) (type default))
-  )
-  (wire (pts (xy 234.95 143.51) (xy 252.095 143.51))
+  (wire (pts (xy 241.3 99.695) (xy 255.27 99.695))
+    (stroke (width 0) (type default))
+  )
+  (wire (pts (xy 234.95 143.51) (xy 241.3 143.51))
     (stroke (width 0) (type default))
   )
@@
     (stroke (width 0) (type default))
   )
+  (wire (pts (xy 193.675 62.23) (xy 193.675 135.89))
+    (stroke (width 0) (type default))
+  )
   (wire (pts (xy 163.83 38.1) (xy 175.26 38.1))
     (stroke (width 0) (type default))
   )
+  (wire (pts (xy 241.3 92.71) (xy 252.095 92.71))
+    (stroke (width 0) (type default))
+  )
   (wire (pts (xy 255.27 138.43) (xy 255.27 150.495))
     (stroke (width 0) (type default))
@@
     (stroke (width 0) (type default))
   )
-  (wire (pts (xy 243.205 145.415) (xy 243.205 150.495))
+  (wire (pts (xy 241.3 145.415) (xy 241.3 150.495))
     (stroke (width 0) (type default))
   )
@@
     (stroke (width 0) (type default))
   )
-  (wire (pts (xy 243.205 94.615) (xy 243.205 99.695))
+  (wire (pts (xy 241.3 94.615) (xy 241.3 99.695))
     (stroke (width 0) (type default))
   )
@@
     (stroke (width 0) (type default))
   )
-  (wire (pts (xy 234.95 145.415) (xy 243.205 145.415))
+  (wire (pts (xy 234.95 145.415) (xy 241.3 145.415))
     (stroke (width 0) (type default))
   )
@@
     )
   )
-  (sheet (at 210.82 29.845) (size 19.685 11.43) (fields_autoplaced)
+  (sheet (at 198.755 29.21) (size 19.685 40.005) (fields_autoplaced)
     (stroke (width 0.1524) (type solid))
     (fill (color 0 0 0 0.0000))
-    (property "Sheetname" "VU_Meter" (at 210.82 29.1334 0)
+    (property "Sheetname" "VU_Meter" (at 198.755 28.4984 0)
       (effects (font (size 1.27 1.27)) (justify left bottom))
     )
-    (property "Sheetfile" "VU-Meter.kicad_sch" (at 210.82 41.8596 0)
+    (property "Sheetfile" "VU-Meter.kicad_sch" (at 198.755 69.7996 0)
       (effects (font (size 1.27 1.27)) (justify left top))
     )
-    (instances
+    (pin "Right" input (at 198.755 62.23 180)
+      (effects (font (size 1.27 1.27)) (justify left))
+    )
+    (pin "5V" input (at 198.755 32.385 180)
+      (effects (font (size 1.27 1.27)) (justify left))
+    )
+    (pin "GND" input (at 198.755 34.29 180)
+      (effects (font (size 1.27 1.27)) (justify left))
+    )
+    (pin "Left" input (at 198.755 64.135 180)
+      (effects (font (size 1.27 1.27)) (justify left))
+    )
+    (instances

Commit message: Reviews, Gerber Plots and Overview Update
Other:
- note added: "Prim"
- note added: "Sek 1"
Changed lines of the file:
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@@
     (stroke (width 0) (type default))
+  )
+  (text "Prim" (at 118.11 177.165 0)
+    (effects (font (size 1.27 1.27)) (justify left bottom))
+  )
+  (text "Sek 1" (at 102.87 70.485 0)
+    (effects (font (size 1.27 1.27)) (justify left bottom))
+  )
+  (text "Prim" (at 118.11 76.835 0)
+    (effects (font (size 1.27 1.27)) (justify left bottom))
+  )
+  (text "Sek 1" (at 102.87 170.815 0)
+    (effects (font (size 1.27 1.27)) (justify left bottom))
+  )
+  (text "Sek 1" (at 102.87 83.185 0)
+    (effects (font (size 1.27 1.27)) (justify left bottom))
+  )
+  (text "Sek 1" (at 102.87 183.515 0)
+    (effects (font (size 1.27 1.27)) (justify left bottom))
   )
   (symbol (lib_id "Connector:Conn_Coaxial") (at 261.62 92.71 0) (unit 1)
@@
   )
   (symbol (lib_id "Device:Transformer_1P_2S") (at 112.395 176.53 0) (mirror y) (unit 1)
-    (in_bom yes) (on_board yes) (dnp no) (fields_autoplaced)
-    (property "Reference" "T8" (at 112.395 162.3526 0)
+    (in_bom yes) (on_board yes) (dnp no)
+    (property "Reference" "T8" (at 112.395 160.655 0)
       (effects (font (size 1.27 1.27)))
     )
-    (property "Value" "2x 45V 600VA" (at 112.395 164.7768 0)
+    (property "Value" "2x 45V 600VA" (at 112.395 162.56 0)
       (effects (font (size 1.27 1.27)))
     )
@@
   )
   (symbol (lib_id "Device:Transformer_1P_2S") (at 112.395 76.2 0) (mirror y) (unit 1)
-    (in_bom yes) (on_board yes) (dnp no) (fields_autoplaced)
-    (property "Reference" "T7" (at 112.395 62.0226 0)
+    (in_bom yes) (on_board yes) (dnp no)
+    (property "Reference" "T7" (at 112.395 60.325 0)
       (effects (font (size 1.27 1.27)))
     )
-    (property "Value" "2x 45V 600VA" (at 112.395 64.4468 0)
+    (property "Value" "2x 45V 600VA" (at 112.395 62.865 0)
       (effects (font (size 1.27 1.27)))
     )

Commit message: Readme and Overview Update
Parts:
- added RV101: 100k log, symbol Device:R_Potentiometer_Dual_Separate
Connections:
- net Channel_2/spk_gnd is gone; now on net Channel_1/spk_gnd: J19.2 (Ext), J20.2 (Ext), J21.2 (Ext), R96.1
- net Channel_1/In_Gnd: now also RV101.3, RV101.6
- net Channel_1/In_Sig: now also RV101.5
- net Channel_2/In_Sig: now also RV101.2
- new net Digitalteil/Left: RV101.4
- new net Digitalteil/Right: RV101.1
Other:
- sheet VU_Meter ports: added Left_Gnd, Right_Gnd; removed none
- note added: "Volume Control"
