File: Hardware/Black_Devil/VU-Meter.kicad_sch (KiCad schematic)
At the start: 151 parts, among them J101 Left, J102 Right, J103 Right, U101 LM2902, U102 LM2902, U103 LM2902, U104 LM2902, U105 LM2902, U106 LM2902, U107 LM2902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

Commit message: Major Update
Repo Cleanup
Finished VU Meter PCB
Finalized Softstart PCB
Finalized Channel PCB
Connections:
- net +5VA: now also J102.2 (Pin_2), U105.6 (-); no longer J102.1 (Pin_1), U105.2 (-)
- net GND: now also J102.1 (Pin_1), J103.1 (Pin_1); no longer J102.2 (Pin_2), J103.2 (Pin_2)
- net at R155.2, R156.2: now also U106.6 (-); no longer U106.2 (-)
- net at R151.2, R152.2: now also U105.13 (-); no longer U105.9 (-)
- net at D126.2 (A): now also U106.1; no longer U106.7
- net at R171.2, R175.1: now also U108.2 (-); no longer U108.6 (-)
- net at R175.2, R176.1: now also U108.13 (-); no longer U108.9 (-)
- net at R161.2, R162.2: now also U106.9 (-); no longer U106.13 (-)
- net at R166.2, R174.2: now also U107.13 (-); no longer U107.9 (-)
- net Left: now reaches D101.2 (A), J101.1 (Pin_1)
- net at U107.1: now also D130.2 (A); no longer D129.2 (A)
- net at R163.2, R164.2: now also U107.6 (-); no longer U107.2 (-)
- net at D134.2 (A): now also U108.1; no longer U108.7
- net at D121.2 (A): now also U105.7; no longer U105.1
- net Right: now reaches D119.2 (A)
- net Right: now also J103.2 (Pin_2); no longer J103.1 (Pin_1)
- net at D133.2 (A): now also U108.7; no longer U108.1
- net at R169.2, R170.2: now also U108.6 (-); no longer U108.2 (-)
- net at R167.2, R168.2: now also U107.9 (-); no longer U107.13 (-)
- net at U107.14: now also D131.2 (A); no longer D132.2 (A)
- net at R159.2, R160.2: now also U106.13 (-); no longer U106.9 (-)
- net at U107.7: now also D129.2 (A); no longer D130.2 (A)
- net at D128.2 (A): now also U106.8; no longer U106.14
- net at D135.2 (A): now also U108.14; no longer U108.8
- net at R157.2, R158.2: now also U106.2 (-); no longer U106.6 (-)
- net at D122.2 (A): now also U105.1; no longer U105.7
- net at R149.2, R150.2: now also U105.2 (-); no longer U105.6 (-)
- net at U107.8: now also D132.2 (A); no longer D131.2 (A)
- net at D136.2 (A): now also U108.8; no longer U108.14
- net at D127.2 (A): now also U106.14; no longer U106.8
- net at R165.2, R174.1: now also U107.2 (-); no longer U107.6 (-)
- net at D125.2 (A): now also U106.7; no longer U106.1
- net at D124.2 (A): now also U105.8; no longer U105.14
- net at R172.2, R176.2: now also U108.9 (-); no longer U108.13 (-)
- net at R153.2, R154.2: now also U105.9 (-); no longer U105.13 (-)
- net at D123.2 (A): now also U105.14; no longer U105.8
Other:
- moved on the sheet: U105A, U105B, U105C, U105D, U106A, U106B, U106C, U106D, U107A, U107B, U107C, U107D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

Commit message: Finalize all PCBs
Connections:
- net GND: now also RV101.3, RV102.1; no longer RV101.1, RV102.3
- net at C108.1, R147.2: now also RV102.3; no longer RV102.1
- net at C103.1, R101.2: now also RV101.1; no longer RV101.3
Changed lines of the file:
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@@
     )
   )
-  (symbol (lib_id "Device:R_Potentiometer_Trim") (at 137.16 28.575 0) (unit 1)
-    (in_bom yes) (on_board yes) (dnp no)
-    (property "Reference" "RV102" (at 135.3821 27.3629 0)
+  (symbol (lib_id "Device:R_Potentiometer_Trim") (at 137.16 28.575 0) (mirror x) (unit 1)
+    (in_bom yes) (on_board yes) (dnp no)
+    (property "Reference" "RV102" (at 135.3821 29.7871 0)
       (effects (font (size 1.27 1.27)) (justify right))
     )
-    (property "Value" "10k" (at 135.3821 29.7871 0)
+    (property "Value" "10k" (at 135.3821 27.3629 0)
       (effects (font (size 1.27 1.27)) (justify right))
     )
@@
     )
   )
-  (symbol (lib_id "Device:R_Potentiometer_Trim") (at 44.45 28.575 0) (mirror x) (unit 1)
-    (in_bom yes) (on_board yes) (dnp no)
-    (property "Reference" "RV101" (at 42.6721 29.7871 0)
+  (symbol (lib_id "Device:R_Potentiometer_Trim") (at 44.45 28.575 0) (unit 1)
+    (in_bom yes) (on_board yes) (dnp no)
+    (property "Reference" "RV101" (at 42.6721 27.3629 0)
       (effects (font (size 1.27 1.27)) (justify right))
     )
-    (property "Value" "10k" (at 42.6721 27.3629 0)
+    (property "Value" "10k" (at 42.6721 29.7871 0)
       (effects (font (size 1.27 1.27)) (justify right))
     )

Commit message: Readme and Overview Update
Changed lines of the file:
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@@
   (junction (at 142.24 59.69) (diameter 0) (color 0 0 0 0)
   )
+  (junction (at 110.49 17.78) (diameter 0) (color 0 0 0 0)
+  )
   (junction (at 145.415 28.575) (diameter 0) (color 0 0 0 0)
   )
@@
   (junction (at 153.035 240.665) (diameter 0) (color 0 0 0 0)
   )
+  (junction (at 18.415 17.78) (diameter 0) (color 0 0 0 0)
+  )
   (junction (at 171.45 221.615) (diameter 0) (color 0 0 0 0)
   )
@@
     (stroke (width 0) (type default))
   )
-  (wire (pts (xy 15.875 17.78) (xy 19.05 17.78))
+  (wire (pts (xy 15.875 17.78) (xy 18.415 17.78))
     (stroke (width 0) (type default))
   )
@@
     (stroke (width 0) (type default))
   )
+  (wire (pts (xy 110.49 20.955) (xy 110.49 17.78))
+    (stroke (width 0) (type default))
+  )
   (wire (pts (xy 44.45 21.59) (xy 33.655 21.59))
     (stroke (width 0) (type default))
@@
     (stroke (width 0) (type default))
   )
+  (wire (pts (xy 18.415 20.955) (xy 18.415 17.78))
+    (stroke (width 0) (type default))
+  )
   (wire (pts (xy 60.325 238.76) (xy 60.325 240.665))
     (stroke (width 0) (type default))
@@
     (stroke (width 0) (type default))
   )
+  (wire (pts (xy 18.415 17.78) (xy 19.05 17.78))
+    (stroke (width 0) (type default))
+  )
   (wire (pts (xy 48.26 127) (xy 49.53 127))
     (stroke (width 0) (type default))
@@
     (stroke (width 0) (type default))
   )
+  (wire (pts (xy 110.49 17.78) (xy 111.76 17.78))
+    (stroke (width 0) (type default))
+  )
   (wire (pts (xy 132.08 157.48) (xy 132.08 154.94))
     (stroke (width 0) (type default))
@@
     (stroke (width 0) (type default))
   )
+  (wire (pts (xy 111.76 20.955) (xy 110.49 20.955))
+    (stroke (width 0) (type default))
+  )
   (wire (pts (xy 49.53 69.85) (xy 53.975 69.85))
     (stroke (width 0) (type default))
@@
     (stroke (width 0) (type default))
   )
-  (wire (pts (xy 108.585 17.78) (xy 111.76 17.78))
+  (wire (pts (xy 108.585 17.78) (xy 110.49 17.78))
     (stroke (width 0) (type default))
   )
@@
     (stroke (width 0) (type default))
   )
+  (wire (pts (xy 19.685 20.955) (xy 18.415 20.955))
+    (stroke (width 0) (type default))
+  )
   (wire (pts (xy 48.26 116.84) (xy 49.53 116.84))
     (stroke (width 0) (type default))
@@
   (wire (pts (xy 142.24 63.5) (xy 142.24 59.69))
     (stroke (width 0) (type default))
+  )
+  (hierarchical_label "Right_Gnd" (shape input) (at 111.76 20.955 0) (fields_autoplaced)
+    (effects (font (size 1.27 1.27)) (justify left))
   )
   (hierarchical_label "5V" (shape input) (at 71.12 260.35 180) (fields_autoplaced)
     (effects (font (size 1.27 1.27)) (justify right))
   )
+  (hierarchical_label "Left_Gnd" (shape input) (at 19.685 20.955 0) (fields_autoplaced)
+    (effects (font (size 1.27 1.27)) (justify left))
+  )
   (hierarchical_label "Right" (shape input) (at 107.315 33.02 0) (fields_autoplaced)
